Commit message: commit from VM

File: annin_ar4_description/urdf/ar_macro.xacro (robot description, xacro)
@@ -162,5 +162,5 @@
     <origin xyz="0 0 -0.00887" rpy="3.14 0 0"/>
     <geometry>
-      <mesh filename="package://annin_ar4_description/meshes/${robot_parameters['mesh_dir']}/Link_2_Col.STL"/>
+      <mesh filename="package://annin_ar4_description/meshes/${robot_parameters['mesh_dir']}/link_2_Col.STL"/>
     </geometry>
   </collision>
@@ -195,5 +195,5 @@
     <origin xyz="0 0 -0.00887" rpy="3.14 0 0"/>
     <geometry>
-      <mesh filename="package://annin_ar4_description/meshes/${robot_parameters['mesh_dir']}/Link_2_Cover.STL"/>
+      <mesh filename="package://annin_ar4_description/meshes/${robot_parameters['mesh_dir']}/link_2_Cover.STL"/>
     </geometry>
     <material name="link2_cover_mat">
@@ -213,5 +213,5 @@
     <origin xyz="0 0 -0.00887" rpy="3.14 0 0"/>
     <geometry>
-      <mesh filename="package://annin_ar4_description/meshes/${robot_parameters['mesh_dir']}/Link_2_Logo.STL"/>
+      <mesh filename="package://annin_ar4_description/meshes/${robot_parameters['mesh_dir']}/link_2_Logo.STL"/>
     </geometry>
     <material name="link2_logo_mat">
@@ -262,5 +262,5 @@
     <origin xyz="0 0 -0.03671" rpy="0 0 0"/>
     <geometry>
-      <mesh filename="package://annin_ar4_description/meshes/${robot_parameters['mesh_dir']}/Link_3_Col.STL"/>
+      <mesh filename="package://annin_ar4_description/meshes/${robot_parameters['mesh_dir']}/link_3_Col.STL"/>
     </geometry>
   </collision>
@@ -325,5 +325,5 @@
     <origin xyz="0 0 -0.07594" rpy="0 0 -1.5708"/>
     <geometry>
-      <mesh filename="package://annin_ar4_description/meshes/${robot_parameters['mesh_dir']}/Link_4_Col.STL"/>
+      <mesh filename="package://annin_ar4_description/meshes/${robot_parameters['mesh_dir']}/link_4_Col.STL"/>
     </geometry>
   </collision>
@@ -423,5 +423,5 @@
     <origin xyz="0 0 -0.0275" rpy="0 0 0"/>
     <geometry>
-      <mesh filename="package://annin_ar4_description/meshes/${robot_parameters['mesh_dir']}/Link_5_Col.STL"/>
+      <mesh filename="package://annin_ar4_description/meshes/${robot_parameters['mesh_dir']}/link_5_Col.STL"/>
     </geometry>
   </collision>
@@ -483,5 +483,5 @@
     <origin xyz="0 0 -0.016" rpy="0 0 0"/>
     <geometry>
-      <mesh filename="package://annin_ar4_description/meshes/${robot_parameters['mesh_dir']}/Link_6_Col.STL"/>
+      <mesh filename="package://annin_ar4_description/meshes/${robot_parameters['mesh_dir']}/link_6_Col.STL"/>
     </geometry>
   </collision>
